File: pcb/snorlax.sch (EAGLE design)
At the start: 13 parts, among them IC1 MCP3008

Commit message: Final PCB Schematics, Board Layouts and Gerber Files
Parts:
- added C1: 22uF, SparkFun-Capacitors:CAP1206
- added J10, J11, J9: (no value), SparkFun-Connectors:M03LOCK
- added J8: (no value), SparkFun-Connectors:M05LOCK
- J1, J2: device SparkFun-Connectors:M05LOCK -> SparkFun-Connectors:M03LOCK
- J3: device SparkFun-Connectors:M08LOCK -> SparkFun-Connectors:M05LOCK
- J6, J7: device SparkFun-Connectors:M08LOCK -> SparkFun-Connectors:M03LOCK
Connections:
- net GND: now also C1.2, J1.3, J10.2, J11.3, J2.3, J3.4, J6.3, J8.4, J9.2; no longer J7.1, J7.2, J7.4, J7.5, J7.6, J7.7, J7.8
- net N$1: now also J3.3; no longer J3.8
- net N$2: now also J3.2; no longer J3.7
- net N$3: now also J3.1; no longer J3.6
- net N$4: now also J8.3; no longer J3.5
- net N$5: now also J8.2; no longer J3.4
- net N$6: now also J8.1; no longer J3.3
- net N$7: now also J9.3; no longer J3.2
- net N$8: now also J10.3; no longer J3.1
- net VCC_3.3: now also C1.1, J1.2, J10.1, J11.2, J3.5, J7.2, J8.5, J9.1; no longer J2.1, J2.3, J2.4, J2.5, J6.1, J6.3, J6.4, J6.5, J6.6
- net VCC_5.5: now also J11.1, J2.1, J6.1, J7.1; no longer J1.2, J1.3, J1.4, J1.5, J6.7, J6.8
Other:
- note added: "Accelerometer 1"
- note added: "Accelerometer 2"
- note added: "GPIO Pins from Pi"
- note added: "Microphone 1"
- note added: "Microphone 2"
- note added: "Powers and Ground from Main PCB to Cluster PCBs"
- note added: "Powers and Ground from Pi"
