File: pcb/snorlax_velostat.brd (EAGLE design)
At the start: 37.8 x 29.2 mm, 18 parts, among them IC1 MCP3008

Commit message: Final PCB Schematics, Board Layouts and Gerber Files
Parts:
- added C1: 22uF, SparkFun-Capacitors:1206
- added J1, J10, J2, J3, J6, J7: (no value), SparkFun-Connectors:1X02_LOCK
- J8, J9: device SparkFun-Connectors:1X08_LOCK -> SparkFun-Connectors:1X02_LOCK
- moved R7 28.2 mm to (2.54, 14.0), turned to 270 degrees
- moved J8 14.5 mm to (22.9, 21.6)
- moved R3 3.81 mm to (25.4, 17.8)
- moved R4 3.81 mm to (20.3, 17.8)
- moved R5 3.81 mm to (15.2, 17.8)
- moved R6 3.81 mm to (10.2, 17.8)
- moved J9 3.59 mm to (29.2, 24.1), turned to 90 degrees
- moved R1 1.27 mm to (5.08, 10.2)
- moved R2 1.27 mm to (5.08, 19.1), turned to 270 degrees
Connections:
- net CH1: now also J1.2; no longer J8.8
- net CH2: now also J2.2; no longer J8.7
- net CH3: now also J3.2; no longer J8.6
- net CH4: now also J6.2; no longer J8.5
- net CH5: now also J7.1; no longer J8.4
- net CH6: now also J8.1; no longer J8.3
- net CH7: now also J9.1; no longer J8.2
- net CH8: now also J10.1; no longer J8.1
- net GND: now also C1.2, J1.1, J10.2, J2.1, J3.1, J6.1, J7.2, J8.2; no longer J9.1, J9.3, J9.4, J9.5, J9.6, J9.7, J9.8
- net VCC_3.3: now also C1.1
Routing:
- net GND: track 77.3 -> 110.3 mm, vias 0 -> 2
- net CH6: track 8.62 -> 37.6 mm, vias 0 -> 2
- net CH3: track 12.0 -> 26.3 mm, vias 0 -> 1
- net CH7: track 26.6 -> 40.2 mm, vias 0 -> 1
- net VCC_3.3: track 6.22 -> 18.2 mm
- net CH1: track 26.9 -> 37.6 mm
- net CH2: track 24.1 -> 34.4 mm, vias 1 -> 2
- net CH5: track 7.67 -> 16.9 mm
- net VCC_5.5: track 67.8 -> 63.0 mm, vias 0 -> 3
- net CH8: track 27.2 -> 31.9 mm
Other:
- board size 37.8 x 29.2 mm -> 39 x 29.2 mm
- board text added: "GPIO"
- board text added: "PWR/GND"
- board text added: "Snorlax Velostat"
- board text added: "V1"
- board text added: "V2"
- board text added: "V3"
- board text added: "V4"
- board text added: "V5"
- board text added: "V6"
- board text added: "V7"
- board text added: "V8"
