File: pcb/snorlax_velostat.sch (EAGLE design)
At the start: 18 parts, among them IC1 MCP3008

Commit message: Final PCB Schematics, Board Layouts and Gerber Files
Parts:
- added C1: 22uF, SparkFun-Capacitors:CAP1206
- added J1, J10, J2, J3, J6, J7: (no value), SparkFun-Connectors:M02LOCK
- J8, J9: device SparkFun-Connectors:M08LOCK -> SparkFun-Connectors:M02LOCK
Connections:
- net CH1: now also J1.2; no longer J8.8
- net CH2: now also J2.2; no longer J8.7
- net CH3: now also J3.2; no longer J8.6
- net CH4: now also J6.2; no longer J8.5
- net CH5: now also J7.1; no longer J8.4
- net CH6: now also J8.1; no longer J8.3
- net CH7: now also J9.1; no longer J8.2
- net CH8: now also J10.1; no longer J8.1
- net GND: now also C1.2, J1.1, J10.2, J2.1, J3.1, J6.1, J7.2, J8.2; no longer J9.1, J9.3, J9.4, J9.5, J9.6, J9.7, J9.8
- net VCC_3.3: now also C1.1
Other:
- note added: "GPIO Pins from Pi"
- note added: "Powers and Ground from Main PCB"
- note added: "The 2-pin headers are for the 8 Velostats on this Cluster PCB"
